Commit message: Remove Green Color in xacro, not definiert

File: urdf/simple_robot.urdf.xacro (robot description, xacro)
@@ -42,5 +42,4 @@
                 <sphere radius=".05" />
             </geometry>
-            <material name="green"/>
         </visual>
     </link>

Commit message: Update Gazebo Tags and Link Names
Correction needed to get friction working properly

File: urdf/simple_robot.urdf.xacro (robot description, xacro)
@@ -2,5 +2,5 @@
 <robot name="simple_robot" xmlns:xacro="http://www.ros.org/wiki/xacro">
     <!-- Start of Links - first link must be a non-inertial link -->
-    <link name='base_link'>
+    <link name="base_link">
     </link>
     <link name="chassis">
@@ -9,10 +9,10 @@
             <inertia ixx="0.004" ixy="0.0" ixz="0.0" iyy="0.004" iyz="0.0" izz="0.002"/>
         </inertial>
-        <collision name='collision'>
+        <collision name="chassis">
             <geometry>
                 <box size=".4 .2 .1" />
             </geometry>
         </collision>
-        <visual name='visual'>
+        <visual name="chassis">
             <geometry>
                 <box size=".4 .2 .1" />
@@ -25,16 +25,8 @@
             <inertia ixx="0.004" ixy="0.0" ixz="0.0" iyy="0.004" iyz="0.0" izz="0.002"/>
         </inertial>
-        <collision name='collision'>
+        <collision name="castor">
             <geometry>
                 <sphere radius=".05" />
             </geometry>
-            <surface>
-                <friction>
-                    <ode>
-                        <mu>0</mu>
-                        <mu2>0</mu2>
-                    </ode>
-                </friction>
-            </surface>
         </collision>
         <visual name='visual'>
@@ -50,10 +42,10 @@
         </inertial>
         <pose>0.1 0.13 0.1 0 1.5707 1.5707</pose>
-        <collision name='collision'>
+        <collision name="left_wheel">
             <geometry>
                 <cylinder radius='.1' length='.05'/>
             </geometry>
         </collision>
-        <visual name='visual'>
+        <visual name="left_wheel">
             <geometry>
                 <cylinder radius='.1' length='.05'/>
@@ -67,10 +59,10 @@
         </inertial>
         <pose>0.1 0.13 0.1 0 1.5707 1.5707</pose>
-        <collision name='collision'>
+        <collision name="right_wheel">
             <geometry>
                 <cylinder radius='.1' length='.05'/>
             </geometry>
         </collision>
-        <visual name='visual'>
+        <visual name="right_wheel">
             <geometry>
                 <cylinder radius='.1' length='.05'/>
@@ -152,17 +144,33 @@
   <gazebo reference="chassis">
   	<material>Gazebo/Green</material>
+    	<mu1>.01</mu1>
+    	<mu2>.01</mu2>
+        <fdir1>0.000000 0.000000 0.000000</fdir1>
+        <slip1>1.000000</slip1>
+        <slip2>1.000000</slip2>
   </gazebo>
   <gazebo reference="left_wheel">
-  	<material>Gazebo/Orange</material>
-    <mu1>1</mu1>
-    <mu2>1</mu2>
+    	<material>Gazebo/Orange</material>
+    	<mu1>100000</mu1>
+    	<mu2>100000</mu2>
+        <fdir1>0.000000 0.000000 0.000000</fdir1>
+        <slip1>0.000000</slip1>
+        <slip2>0.000000</slip2>
   </gazebo>
   <gazebo reference="right_wheel">
-  	<material>Gazebo/Orange</material>
-    <mu1>1</mu1>
-    <mu2>1</mu2>
+    	<material>Gazebo/Orange</material>
+    	<mu1>100000</mu1>
+    	<mu2>100000</mu2>
+        <fdir1>0.000000 0.000000 0.000000</fdir1>
+        <slip1>0.000000</slip1>
+        <slip2>0.000000</slip2>
   </gazebo>
   <gazebo reference="castor">
   	<material>Gazebo/Blue</material>
+    	<mu1>.01</mu1>
+    	<mu2>.01</mu2>
+        <fdir1>0.000000 0.000000 0.000000</fdir1>
+        <slip1>1.000000</slip1>
+        <slip2>1.000000</slip2>
   </gazebo>
 </robot>

Commit message: Update Colours

File: urdf/simple_robot.urdf.xacro (robot description, xacro)
@@ -151,5 +151,5 @@
   </gazebo>
   <gazebo reference="left_wheel">
-    	<material>Gazebo/Orange</material>
+    	<material>Gazebo/Red</material>
     	<mu1>100000</mu1>
     	<mu2>100000</mu2>
@@ -159,5 +159,5 @@
   </gazebo>
   <gazebo reference="right_wheel">
-    	<material>Gazebo/Orange</material>
+    	<material>Gazebo/Yellow</material>
     	<mu1>100000</mu1>
     	<mu2>100000</mu2>
